Commit message: (1) Added mesh files in ../urdf/include/meshes/* to avoid dependency on zed-ros-interface; (2) added an extra argument to all launch files called . The argument is a bool value indicating whether zed-nodelet has to start in sim-mode or not.

File: zed_wrapper/urdf/zed_macro.urdf.xacro (robot description, xacro)
@@ -66,5 +66,5 @@
         <origin xyz="${screw_offset_x} 0 0" rpy="0 0 0"/>
         <geometry>
-          <mesh filename="package://zed_interfaces/meshes/${model}.stl" />
+          <mesh filename="file://$(find zed_wrapper)/urdf/include/meshes/${model}.stl" />
         </geometry>
         <material name="${model}_mat" />
@@ -72,5 +72,5 @@
       <collision>
         <geometry>
-          <mesh filename="package://zed_interfaces/meshes/${model}.stl" />
+          <mesh filename="file://$(find zed_wrapper)/urdf/include/meshes/${model}.stl" />
         </geometry>
       </collision>
